Commit message: Dual-arm bases to 18 in apart; full camera suite with customizable globals
- so101_dual_follower.xml + so101_dual.urdf: left/right bases moved from
  y=±0.28 to ±0.2286 (18 in = 0.4572 m base separation, Z/X axes parallel —
  matches the real rig); README notes updated.
- so101.urdf: fix illegal '--' inside XML comment (broke standards-compliant
  parsers, e.g. the Isaac URDF importer).
- Wrist camera XML defaults synced to the tuned env CameraConfig values.
- All 4 task envs gain global overhead_cam (top-down) + front_cam (workspace
  view); front_cam euler fixed everywhere ((0,55,0) pointed away from the
  workspace; (75,0,0) frames it).
- Every camera customizable at runtime via CameraConfig (pos/euler/fov/w/h).
- Per-env camera grid screenshots (images/cameras.png) rendered from the
  live envs post-change; ENVS.md refreshed.

All 6 envs pass --headless-check and zero/random action validation.

File: robots/so101/so101_dual.urdf (robot description, URDF)
Before this commit: robot so101_dual, 17 links, 16 joints
Joints:
- joint left_base_fixed: origin xyz=0.18 0.28 0.82 rpy=0 0 0 -> xyz=0.18 0.2286 0.82 rpy=0 0 0
- joint right_base_fixed: origin xyz=0.18 -0.28 0.82 rpy=0 0 0 -> xyz=0.18 -0.2286 0.82 rpy=0 0 0
